Commit message: A3 asset v2: primitive collisions (fix MJWarp nefc overflow), URDF zero-mass fix (caught by cross-sim comparator), Isaac check script, bootstrap report
Co-Authored-By: Claude Fable 5 <noreply@anthropic.com>

File: assets/a3_ultra/holosoma/a3_ultra_29dof.urdf (robot description, URDF)
Before this commit: robot a3_ultra_29dof, 47 links, 46 joints
Links:
- link D415_in_torso_Link: mass 0 -> 1e-4
- link D457_in_torso_Link: mass 0 -> 1e-4
- link left_knee_shell_Link: mass 0 -> 1e-4
- link right_knee_shell_Link: mass 0 -> 1e-4
- link senyun_in_torso_Link: mass 0 -> 1e-4
- link torso_shell_Link: mass 0 -> 1e-4
- link ultra_head_fisheye_camera_back_Link: mass 0 -> 1e-4
- link ultra_head_fisheye_camera_left_Link: mass 0 -> 1e-4
- link ultra_head_fisheye_camera_right_Link: mass 0 -> 1e-4
- link ultra_head_mid360_Link: mass 0 -> 1e-4
- link ultra_head_stereo_camera_Link: mass 0 -> 1e-4

Commit message: Fix IsaacSim cloud failure: URDF now contains exactly the 34 config bodies (decorative links removed, inertials synced from compiled MJCF, contact-point links added) — importer does not merge fixed joints
Co-Authored-By: Claude Fable 5 <noreply@anthropic.com>

File: assets/a3_ultra/holosoma/a3_ultra_29dof.urdf (robot description, URDF)
Before this commit: robot a3_ultra_29dof, 47 links, 46 joints
Links:
- removed link D415_in_torso_Link
- removed link D457_in_torso_Link
- removed link imu_in_pelvis_Link
- removed link imu_in_torso_Link
- removed link left_hand_palm_Link
- removed link left_knee_shell_Link
- removed link right_hand_palm_Link
- removed link right_knee_shell_Link
- removed link senyun_in_torso_Link
- removed link torso_shell_Link
- removed link ultra_head_fisheye_camera_back_Link
- removed link ultra_head_fisheye_camera_left_Link
- removed link ultra_head_fisheye_camera_right_Link
- removed link ultra_head_mid360_Link
- removed link ultra_head_stereo_camera_Link
- added link left_foot_contact_point, mass 0.001; visual box size=0.001 0.001 0.001
- added link right_foot_contact_point, mass 0.001; visual box size=0.001 0.001 0.001
- link head_pitch_Link: mass 1.672 -> 1.67200000; geometry collision box size=0.159252 0.199156 0.241246; visual mesh filename=meshes/ultra_head_pitch_Link.STL
- link head_yaw_Link: mass 0.8 -> 0.80000000; geometry collision box size=0.111670 0.141578 0.191894; visual mesh filename=meshes/head_yaw_Link.STL
- link left_ankle_pitch_Link: mass 0.10100813 -> 0.10100800; geometry visual mesh filename=meshes/left_ankle_pitch_Link.STL
- link left_ankle_roll_Link: mass 0.82544987 -> 0.82545000; geometry collision sphere radius=0.002000; collision sphere radius=0.002000
- link left_elbow_Link: mass 0.71204442 -> 0.71204400; geometry collision box size=0.082608 0.089270 0.180078; visual mesh filename=meshes/left_elbow_Link.STL
- link left_hip_pitch_Link: mass 1.87345917 -> 1.87346000; geometry collision box size=0.136778 0.128344 0.188032; visual mesh filename=meshes/left_hip_pitch_Link.STL
- link left_hip_roll_Link: mass 0.74493005 -> 0.74493000; geometry collision box size=0.142962 0.141496 0.142898; visual mesh filename=meshes/left_hip_roll_Link.STL
- link left_hip_yaw_Link: mass 2.64563497 -> 2.64563000; geometry collision box size=0.148476 0.144928 0.339008; visual mesh filename=meshes/left_hip_yaw_Link.STL
- link left_knee_Link: mass 5.23624455 -> 5.23624000; geometry collision box size=0.114258 0.144202 0.494902; visual mesh filename=meshes/left_knee_Link.STL
- link left_shoulder_pitch_Link: mass 1.01944747 -> 1.01945000; geometry visual mesh filename=meshes/left_shoulder_pitch_Link.STL
- link left_shoulder_roll_Link: mass 0.95854774 -> 0.95854800; geometry collision box size=0.100112 0.122044 0.195834; visual mesh filename=meshes/left_shoulder_roll_Link.STL
- link left_shoulder_yaw_Link: mass 0.99955871 -> 0.99955900; geometry collision box size=0.096814 0.099818 0.174710; visual mesh filename=meshes/left_shoulder_yaw_Link.STL
- link left_wrist_pitch_Link: mass 0.56746364 -> 0.56746400; geometry collision box size=0.053994 0.054000 0.100006; visual mesh filename=meshes/left_wrist_pitch_Link.STL
- link left_wrist_roll_Link: mass 0.19185994 -> 0.19186000; geometry collision box size=0.074844 0.075322 0.075984; visual mesh filename=meshes/left_wrist_roll_Link.STL
- link left_wrist_yaw_Link: mass 0.08067756 -> 0.53932300; geometry collision box size=0.055996 0.076186 0.074172; collision box size=0.087252 0.090200 0.129314
- link pelvis_link: mass 4.98224861 -> 5.00225000; geometry collision box size=0.161664 0.175468 0.199530; visual mesh filename=meshes/pelvis_link.STL
- link right_ankle_pitch_Link: mass 0.10100813 -> 0.10100800; geometry visual mesh filename=meshes/right_ankle_pitch_Link.STL
- link right_ankle_roll_Link: mass 0.82544987 -> 0.82545000; geometry collision sphere radius=0.002000; collision sphere radius=0.002000
- link right_elbow_Link: mass 0.71187773 -> 0.71187800; geometry collision box size=0.082610 0.089270 0.180080; visual mesh filename=meshes/right_elbow_Link.STL
- link right_hip_pitch_Link: mass 1.87346368 -> 1.87346000; geometry collision box size=0.136778 0.128344 0.188108; visual mesh filename=meshes/right_hip_pitch_Link.STL
- link right_hip_roll_Link: mass 0.74491385 -> 0.74491400; geometry collision box size=0.142962 0.141498 0.142904; visual mesh filename=meshes/right_hip_roll_Link.STL
- link right_hip_yaw_Link: mass 2.6488815 -> 2.64888000; geometry collision box size=0.148148 0.144970 0.338892; visual mesh filename=meshes/right_hip_yaw_Link.STL
- link right_knee_Link: mass 5.23155146 -> 5.23155000; geometry collision box size=0.114258 0.144140 0.494904; visual mesh filename=meshes/right_knee_Link.STL
- link right_shoulder_pitch_Link: mass 1.0194192 -> 1.01942000; geometry visual mesh filename=meshes/right_shoulder_pitch_Link.STL
- link right_shoulder_roll_Link: mass 0.95852346 -> 0.95852300; geometry collision box size=0.100078 0.122044 0.195834; visual mesh filename=meshes/right_shoulder_roll_Link.STL
- link right_shoulder_yaw_Link: mass 0.99859942 -> 0.99859900; geometry collision box size=0.096814 0.099720 0.174630; visual mesh filename=meshes/right_shoulder_yaw_Link.STL
- link right_wrist_pitch_Link: mass 0.56746364 -> 0.56746400; geometry collision box size=0.054000 0.054000 0.099996; visual mesh filename=meshes/right_wrist_pitch_Link.STL
- link right_wrist_roll_Link: mass 0.19185994 -> 0.19186000; geometry collision box size=0.074834 0.075320 0.075984; visual mesh filename=meshes/right_wrist_roll_Link.STL
- link right_wrist_yaw_Link: mass 0.08067756 -> 0.53921600; geometry collision box size=0.055996 0.076186 0.074172; collision box size=0.086972 0.090802 0.129598
- link torso_Link: mass 19.47561404 -> 19.49560000; geometry collision box size=0.295608 0.292964 0.445584; visual mesh filename=meshes/torso_Link.STL
- link waist_roll_Link: mass 0.13538217 -> 0.13538200; geometry visual mesh filename=meshes/waist_roll_Link.STL
- link waist_yaw_Link: mass 0.24519419 -> 0.24519400; geometry visual mesh filename=meshes/waist_yaw_Link.STL
Joints:
- removed joint D415_in_torso_joint
- removed joint D457_in_torso_joint
- removed joint imu_in_pelvis_joint
- removed joint imu_in_torso_joint
- removed joint left_hand_palm_joint
- removed joint left_knee_shell_joint
- removed joint right_hand_palm_joint
- removed joint right_knee_shell_joint
- removed joint senyun_in_torso_joint
- removed joint torso_shell_joint
- removed joint ultra_head_fisheye_camera_back_joint
- removed joint ultra_head_fisheye_camera_left_joint
- removed joint ultra_head_fisheye_camera_right_joint
- removed joint ultra_head_mid360_joint
- removed joint ultra_head_stereo_camera_joint
- added joint left_foot_contact_point_joint: type fixed, parent left_ankle_roll_Link, child left_foot_contact_point, origin xyz=0.04 0 -0.067 rpy=0 0 0
- added joint right_foot_contact_point_joint: type fixed, parent right_ankle_roll_Link, child right_foot_contact_point, origin xyz=0.04 0 -0.067 rpy=0 0 0
